File: soil_moisture.kicad_pcb (KiCad board)
At the start: 2 copper layers, 66.5 x 65 mm, 9 parts, among them J1 Conn_01x03_Pin, J2 Conn_01x02_Pin, K1 Relay_SPDT, M1 Motor_DC, Q1 BC547

Commit message: Initial commit with KiCad project and fabrication files
Routing:
- net +12V: track 135.9 -> 135.3 mm
Changed lines of the file:
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@@
 			(outputformat 1)
 			(mirror no)
-			(drillshape 1)
+			(drillshape 0)
 			(scaleselection 1)
-			(outputdirectory "")
+			(outputdirectory "C:/Users/Susan/Documents/soil_moisture/soil_drill_files")
 		)
 	)
@@
 	)
 	(segment
-		(start 140.5 83.5)
-		(end 140.5 93.5)
+		(start 132 93.5)
+		(end 139.5 93.5)
 		(width 0.2)
 		(layer "B.Cu")
@@
 	)
 	(segment
-		(start 140.5 93.5)
-		(end 132 93.5)
+		(start 141.5 82.5)
+		(end 140.5 83.5)
 		(width 0.2)
 		(layer "B.Cu")
@@
 	)
 	(segment
-		(start 141.5 82.5)
-		(end 140.5 83.5)
+		(start 132 93.5)
+		(end 131 92.5)
 		(width 0.2)
 		(layer "B.Cu")
@@
 	)
 	(segment
-		(start 132 93.5)
-		(end 131 92.5)
+		(start 139.5 93.5)
+		(end 140.5 92.5)
+		(width 0.2)
+		(layer "B.Cu")
+		(net 31)
+	)
+	(segment
+		(start 140.5 92.5)
+		(end 140.5 83.5)
 		(width 0.2)
 		(layer "B.Cu")
